File: LED Wheel/LED_Controller.sch (KiCad schematic (older format))
At the start: 79 parts, among them U1 AZ1117-3.3, U2 PCA9745, U3 PCA9745, U4 PCA9745, U5 PCA9745

Commit message: Init Commit
Initial Commit with the Near-Finished Board Layout
Parts:
- removed D10, D16, D2, D25, D27, D29, D42, D57: G_LED, LED_SMD:LED_0805_2012Metric_Pad1.15x1.40mm_HandSolder, symbol Device:LED
- added D? (x8): R_LED, LED_SMD:LED_0805_2012Metric_Pad1.15x1.40mm_HandSolder, symbol Device:LED
- D?: renamed from D1; value G_LED -> R_LED
- D?: renamed from D26; value G_LED -> R_LED
- D?: renamed from D18; value G_LED -> R_LED
- D?: renamed from D3; value G_LED -> R_LED
- D?: renamed from D28; value G_LED -> R_LED
- D?: renamed from D21; value G_LED -> R_LED
- D?: renamed from D13; value G_LED -> R_LED
- D?: renamed from D5; value G_LED -> R_LED
- D?: renamed from D30; value G_LED -> R_LED
- D?: renamed from D22; value G_LED -> R_LED
- D?: renamed from D32; value G_LED -> R_LED
- D?: renamed from D49; value G_LED -> R_LED
- D?: renamed from D50; value G_LED -> R_LED
- D?: renamed from D53; value G_LED -> R_LED
- D?: renamed from D45; value G_LED -> R_LED
- D?: renamed from D17; value G_LED -> R_LED
- D?: renamed from D9; value G_LED -> R_LED
- D?: renamed from D19; value G_LED -> R_LED
- D?: renamed from D11; value G_LED -> R_LED
- D?: renamed from D20; value G_LED -> R_LED
- D?: renamed from D12; value G_LED -> R_LED
- D?: renamed from D4; value G_LED -> R_LED
- D?: renamed from D14; value G_LED -> R_LED
- D?: renamed from D6; value G_LED -> R_LED
- D?: renamed from D31; value G_LED -> R_LED
- D?: renamed from D23; value G_LED -> R_LED
- D?: renamed from D15; value G_LED -> R_LED
- D?: renamed from D7; value G_LED -> R_LED
- D?: renamed from D24; value G_LED -> R_LED
- D?: renamed from D8; value G_LED -> R_LED
- D?: renamed from D41; value G_LED -> R_LED
- D?: renamed from D33; value G_LED -> R_LED
- D?: renamed from D58; value G_LED -> R_LED
- D?: renamed from D34; value G_LED -> R_LED
- D?: renamed from D59; value G_LED -> R_LED
- D?: renamed from D51; value G_LED -> R_LED
- D?: renamed from D43; value G_LED -> R_LED
- D?: renamed from D35; value G_LED -> R_LED
- D?: renamed from D60; value G_LED -> R_LED
- D?: renamed from D52; value G_LED -> R_LED
- D?: renamed from D44; value G_LED -> R_LED
- D?: renamed from D36; value G_LED -> R_LED
- D?: renamed from D61; value G_LED -> R_LED
- D?: renamed from D37; value G_LED -> R_LED
- D?: renamed from D62; value G_LED -> R_LED
- D?: renamed from D54; value G_LED -> R_LED
- D?: renamed from D46; value G_LED -> R_LED
- D?: renamed from D38; value G_LED -> R_LED
- D?: renamed from D63; value G_LED -> R_LED
- D?: renamed from D55; value G_LED -> R_LED
- D?: renamed from D47; value G_LED -> R_LED
- D?: renamed from D39; value G_LED -> R_LED
- D?: renamed from D64; value G_LED -> R_LED
- D?: renamed from D56; value G_LED -> R_LED
- D?: renamed from D48; value G_LED -> R_LED
- D?: renamed from D40; value G_LED -> R_LED
- renumbered C4 to C?, C3 to C?, C5 to C?, C6 to C?, C1 to C?, C2 to C?, R4 to R?, R1 to R?, R2 to R?, R3 to R?, U2 to U?, U3 to U?, U4 to U?, U5 to U?, U1 to U?
Connections:
- net at U?.13 (LED6): now also D?.1 (K) (x2)
- net at U?.14 (LED7): now also D?.1 (K)
- net at U?.15 (LED8): now also D?.1 (K)
- net at U?.6 (LED0): now also D?.1 (K) (x3)
- net at U?.22 (LED14): now also D?.1 (K)
- net G_12V renamed +12V
- net +12V: now also D?.2 (A), D?.2 (A), D?.2 (A), D?.2 (A), D?.2 (A), D?.2 (A), D?.2 (A), D?.2 (A)
- net G_3V3 renamed +3V3
- net ~CS~_GREEN renamed ~CS~_RED
