File: LED Wheel/B_LED_Controller.sch (KiCad schematic (older format))
At the start: 76 parts

Commit message: Init Commit
Initial Commit with the Near-Finished Board Layout
Parts:
- removed C? (x4): 100N, Capacitor_SMD:C_0603_1608Metric_Pad1.08x0.95mm_HandSolder, symbol Device:C
- removed D? (x36): B_LED, LED_SMD:LED_0805_2012Metric_Pad1.15x1.40mm_HandSolder, symbol Device:LED
- removed R? (x2): 3K, Resistor_SMD:R_1206_3216Metric_Pad1.30x1.75mm_HandSolder, symbol Device:R
- removed U?: PCA9745, Package_SO:HTSSOP-28-1EP_4.4x9.7mm_P0.65mm_EP2.85x5.4mm, symbol Project_Library:PCA9745
- added C13: 10U, Capacitor_SMD:C_0603_1608Metric_Pad1.08x0.95mm_HandSolder, symbol Device:C
- added C14: 22U, Capacitor_SMD:C_0603_1608Metric_Pad1.08x0.95mm_HandSolder, symbol Device:C
- added C15, C16, C17, C18: 100N, Capacitor_SMD:C_0603_1608Metric_Pad1.08x0.95mm_HandSolder, symbol Device:C
- added D132, D135, D136, D137, D139, D140, D151, D153, D154, D155, D156, D157, D158, D159, D160, D162, D163, D164, D165, D166, D167, D168, D169, D171, D172, D174, D176, D178, D180, D183, D184, D185, D186, D187, D188, D192: B_LED, LED_SMD:LED_0805_2012Metric_Pad1.15x1.40mm_HandSolder, symbol Device:LED
- added R12, R9: 3K, Resistor_SMD:R_1206_3216Metric_Pad1.30x1.75mm_HandSolder, symbol Device:R
- added U11: AZ1117-3.3, Package_TO_SOT_SMD:SOT-89-3_Handsoldering, symbol Regulator_Linear:AZ1117-3.3
- added U13: PCA9745, Package_SO:HTSSOP-28-1EP_4.4x9.7mm_P0.65mm_EP2.85x5.4mm, symbol Project_Library:PCA9745
- gave numbers to parts that had none: 33
Connections:
- net EP: now also C13.2, C14.2, C15.2, C16.2, C17.2, C18.2, R12.2, R9.2, U11.1 (GND), U13.10 (VSS), U13.19 (VSS), U13.2 (VSS), U13.24 (VSS), U13.29 (EP)
- net SPI1_CLK: now also U13.26 (SCLK)
- net ~CS~_BLUE: now also U13.4 (~CS~)
- net ~OE~: now also U13.5 (~OE~)
- net ~RESET~: now also U13.25 (~RESET~)
- net at U12.1 (REXT): now also R9.1
- net at U12.11 (LED4): now also D137.1 (K)
- net at U12.12 (LED5): now also D139.1 (K)
- net at U12.18 (LED11): now also D151.1 (K)
- net at U12.20 (LED12): now also D153.1 (K)
- net at U12.21 (LED13): now also D155.1 (K)
- net at U12.22 (LED14): now also D157.1 (K)
- net at U12.23 (LED15): now also D159.1 (K)
- net at U12.9 (LED3): now also D135.1 (K)
- net at U14.11 (LED4): now also D169.1 (K)
- net at U14.12 (LED5): now also D171.1 (K)
- net at U14.18 (LED11): now also D183.1 (K)
- net at U14.20 (LED12): now also D185.1 (K)
- net at U14.21 (LED13): now also D187.1 (K)
- net at U14.3 (SDO): now also U13.27 (SDI)
- net at U14.7 (LED1): now also D163.1 (K)
- net at U14.8 (LED2): now also D165.1 (K)
- net at U14.9 (LED3): now also D167.1 (K)
- net at R10.1: now also U13.1 (REXT)
- net at D138.1 (K): now also U13.11 (LED4)
- net at D142.1 (K): now also U13.13 (LED6)
- net at D144.1 (K): now also U13.14 (LED7)
- net at D146.1 (K): now also U13.15 (LED8)
- net at D148.1 (K): now also U13.16 (LED9)
- net at D150.1 (K): now also U13.17 (LED10)
- net at D152.1 (K): now also U13.18 (LED11)
- net at U15.27 (SDI): now also U13.3 (SDO)
- net at D130.1 (K): now also U13.6 (LED0)
- net at D134.1 (K): now also U13.8 (LED2)
- net at U15.1 (REXT): now also R12.1
- net at U15.12 (LED5): now also D172.1 (K)
- net at U15.13 (LED6): now also D174.1 (K)
- net at U15.14 (LED7): now also D176.1 (K)
- net at U15.15 (LED8): now also D178.1 (K)
- net at U15.16 (LED9): now also D180.1 (K)
- net at U15.18 (LED11): now also D184.1 (K)
- net at U15.20 (LED12): now also D186.1 (K)
- net at U15.21 (LED13): now also D188.1 (K)
- net at U15.23 (LED15): now also D192.1 (K)
- net at U15.6 (LED0): now also D162.1 (K)
- net at U15.7 (LED1): now also D164.1 (K)
- net at U15.8 (LED2): now also D166.1 (K)
- net at U15.9 (LED3): now also D168.1 (K)
- net +12V renamed B_12V
- net B_12V: now also C13.1, D132.2 (A), D135.2 (A), D136.2 (A), D137.2 (A), D139.2 (A), D140.2 (A), D151.2 (A), D153.2 (A), D154.2 (A), D155.2 (A), D156.2 (A), D157.2 (A), D158.2 (A), D159.2 (A), D160.2 (A), D162.2 (A), D163.2 (A), D164.2 (A), D165.2 (A), D166.2 (A), D167.2 (A), D168.2 (A), D169.2 (A), D171.2 (A), D172.2 (A), D174.2 (A), D176.2 (A), D178.2 (A), D180.2 (A), D183.2 (A), D184.2 (A), D185.2 (A), D186.2 (A), D187.2 (A), D188.2 (A), D192.2 (A), U11.3 (VI)
- net +3V3 renamed B_3V3
- net B_3V3: now also C14.1, C15.1, C16.1, C17.1, C18.1, U11.2 (VO), U13.28 (VDD)
- new net: D140.1 (K), U13.12 (LED5)
- new net: D132.1 (K), U13.7 (LED1)
- new net: D154.1 (K), U13.20 (LED12)
- new net: D156.1 (K), U13.21 (LED13)
- new net: D158.1 (K), U13.22 (LED14)
- new net: D160.1 (K), U13.23 (LED15)
- new net: D136.1 (K), U13.9 (LED3)
Other:
- moved on the sheet: D129, D131, D133, D141, D143, D145, D147, D149, D161, D173, D175, D177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

Commit message: Rev A0 Commit
Files all sent to PCB manufacturer & BOM
Connections:
- net SPI1_MISO: now also U12.3 (SDO); no longer U15.3 (SDO)
- net SPI1_MOSI: now also U15.27 (SDI); no longer U12.27 (SDI)
- net at U14.27 (SDI): now also U13.3 (SDO); no longer U12.3 (SDO)
- net at U14.3 (SDO): now also U12.27 (SDI); no longer U13.27 (SDI)
- new net: U13.27 (SDI), U15.3 (SDO)
Changed lines of the file:
@@
 Wire Wire Line
 	3550 1800 3625 1800
-Text HLabel 3550 1900 0    50   Input ~ 0
+Text HLabel 7850 4650 0    50   Input ~ 0
 SPI1_MOSI
-Wire Wire Line
-	3550 1900 3625 1900
 Text HLabel 3550 2100 0    50   Input ~ 0
 SPI1_CLK
@@
 	7925 4950 7850 4950
 Wire Wire Line
-	3625 2000 2550 2000
-Wire Wire Line
-	2550 2000 2550 4650
-Wire Wire Line
-	2550 4650 3625 4650
-Wire Wire Line
-	3625 4750 2550 4750
-Wire Wire Line
-	2550 4750 2550 6500
-Wire Wire Line
 	2550 6500 6350 6500
 Wire Wire Line
-	6350 6500 6350 1900
-Wire Wire Line
-	6350 1900 7925 1900
-Wire Wire Line
-	7925 2000 6650 2000
-Wire Wire Line
-	6650 2000 6650 4650
-Wire Wire Line
-	7925 4650 6650 4650
-Text HLabel 7850 4750 0    50   Output ~ 0
+	6350 6500 6350 2000
+Text HLabel 3625 2000 0    50   Output ~ 0
 SPI1_MISO
-Wire Wire Line
-	7850 4750 7925 4750
 $Comp
 L Regulator_Linear:AZ1117-3.3 U11
@@
 Wire Wire Line
 	8300 5925 8300 6200
+Wire Wire Line
+	7850 4650 7925 4650
+Wire Wire Line
+	6650 4750 7925 4750
+Wire Wire Line
+	6650 1900 7925 1900
+Wire Wire Line
+	6650 1900 6650 4750
+Wire Wire Line
+	7925 2000 6350 2000
+Wire Wire Line
+	3625 4650 2550 4650
+Wire Wire Line
+	2550 4650 2550 6500
+Wire Wire Line
+	3625 4750 2450 4750
+Wire Wire Line
+	2450 4750 2450 1900
+Wire Wire Line
+	2450 1900 3625 1900
 $EndSCHEMATC
