File: LED Wheel/G_LED_Controller.sch (KiCad schematic (older format))
At the start: 76 parts

Commit message: Init Commit
Initial Commit with the Near-Finished Board Layout
Parts:
- removed D? (x8): R_LED, LED_SMD:LED_0805_2012Metric_Pad1.15x1.40mm_HandSolder, symbol Device:LED
- added C1: 10U, Capacitor_SMD:C_0603_1608Metric_Pad1.08x0.95mm_HandSolder, symbol Device:C
- added C2: 22U, Capacitor_SMD:C_0603_1608Metric_Pad1.08x0.95mm_HandSolder, symbol Device:C
- added D1, D13, D14, D15, D17, D2, D33, D61: G_LED, LED_SMD:LED_0805_2012Metric_Pad1.15x1.40mm_HandSolder, symbol Device:LED
- added U1: AZ1117-3.3, Package_TO_SOT_SMD:SOT-89-3_Handsoldering, symbol Regulator_Linear:AZ1117-3.3
- D10, D11, D12, D16, D18, D19, D20, D21, D22, D23, D24, D25, D26, D27, D28, D29, D3, D30, D31, D32, D34, D35, D36, D37, D38, D39, D4, D40, D41, D42, D43, D44, D45, D46, D47, D48, D49, D5, D50, D51, D52, D53, D54, D55, D56, D57, D58, D59, D6, D60, D62, D63, D64, D7, D8, D9: renamed from D?; value R_LED -> G_LED
- gave numbers to parts that had none: 12
Connections:
- net EP: now also C1.2, C2.2, U1.1 (GND)
- net at U2.6 (LED0): now also D1.1 (K)
- net at U2.13 (LED6): now also D13.1 (K)
- net at U2.14 (LED7): now also D15.1 (K)
- net at U2.15 (LED8): now also D17.1 (K)
- net at U4.6 (LED0): now also D33.1 (K)
- net at U4.22 (LED14): now also D61.1 (K)
- net at U3.6 (LED0): now also D2.1 (K)
- net at U3.13 (LED6): now also D14.1 (K)
- net +12V renamed G_12V
- net G_12V: now also C1.1, D1.2 (A), D13.2 (A), D14.2 (A), D15.2 (A), D17.2 (A), D2.2 (A), D33.2 (A), D61.2 (A), U1.3 (VI)
- net +3V3 renamed G_3V3
- net G_3V3: now also C2.1, U1.2 (VO)
- net ~CS~_RED renamed ~CS~_GREEN
Other:
- moved on the sheet: C3, C5, D11, D19, D21, D23, D25, D27, D29, D3, D31, D35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

Commit message: Rev A0 Commit
Files all sent to PCB manufacturer & BOM
Connections:
- net SPI1_MISO: now also U2.3 (SDO); no longer U5.3 (SDO)
- net SPI1_MOSI: now also U5.27 (SDI); no longer U2.27 (SDI)
- net at U4.27 (SDI): now also U3.3 (SDO); no longer U2.3 (SDO)
- net at U4.3 (SDO): now also U2.27 (SDI); no longer U3.27 (SDI)
- new net: U3.27 (SDI), U5.3 (SDO)
Changed lines of the file:
@@
 Wire Wire Line
 	3575 1800 3650 1800
-Text HLabel 3575 1900 0    50   Input ~ 0
+Text HLabel 7850 4650 0    50   Input ~ 0
 SPI1_MOSI
 Wire Wire Line
-	3575 1900 3650 1900
+	7850 4650 7925 4650
 Text HLabel 3575 2100 0    50   Input ~ 0
 SPI1_CLK
@@
 	7925 4950 7850 4950
 Wire Wire Line
-	3650 2000 2575 2000
-Wire Wire Line
-	2575 2000 2575 4650
-Wire Wire Line
-	2575 4650 3650 4650
-Wire Wire Line
-	3650 4750 2575 4750
-Wire Wire Line
-	2575 4750 2575 6500
-Wire Wire Line
-	2575 6500 6350 6500
-Wire Wire Line
-	6350 6500 6350 1900
-Wire Wire Line
-	6350 1900 7925 1900
-Wire Wire Line
-	7925 2000 6650 2000
-Wire Wire Line
-	6650 2000 6650 4650
-Wire Wire Line
-	7925 4650 6650 4650
-Text HLabel 7850 4750 0    50   Output ~ 0
+	3650 1900 2575 1900
+Wire Wire Line
+	2500 6500 6350 6500
+Wire Wire Line
+	6350 6500 6350 2000
+Wire Wire Line
+	7925 1900 6650 1900
+Wire Wire Line
+	7925 4750 6650 4750
+Text HLabel 3575 2000 0    50   Output ~ 0
 SPI1_MISO
 Wire Wire Line
-	7850 4750 7925 4750
+	3575 2000 3650 2000
 $Comp
 L Regulator_Linear:AZ1117-3.3 U1
@@
 Wire Wire Line
 	8300 5925 8300 6175
+Wire Wire Line
+	6350 2000 7925 2000
+Wire Wire Line
+	6650 1900 6650 4750
+Wire Wire Line
+	2575 4750 3650 4750
+Wire Wire Line
+	2575 1900 2575 4750
+Wire Wire Line
+	3650 4650 2500 4650
+Wire Wire Line
+	2500 4650 2500 6500
 $EndSCHEMATC
