File: LED Wheel/R_LED_Controller.sch (KiCad schematic (older format))
At the start: 76 parts

Commit message: Init Commit
Initial Commit with the Near-Finished Board Layout
Parts:
- removed D? (x20): G_LED, LED_SMD:LED_0805_2012Metric_Pad1.15x1.40mm_HandSolder, symbol Device:LED
- removed R? (x2): 3K, Resistor_SMD:R_1206_3216Metric_Pad1.30x1.75mm_HandSolder, symbol Device:R
- removed U? (x3): PCA9745, Package_SO:HTSSOP-28-1EP_4.4x9.7mm_P0.65mm_EP2.85x5.4mm, symbol Project_Library:PCA9745
- added C7: 10U, Capacitor_SMD:C_0603_1608Metric_Pad1.08x0.95mm_HandSolder, symbol Device:C
- added C8: 22U, Capacitor_SMD:C_0603_1608Metric_Pad1.08x0.95mm_HandSolder, symbol Device:C
- added D106, D109, D111, D113, D115, D117, D118, D126, D127, D67, D69, D70, D74, D80, D82, D83, D84, D85, D86, D88: R_LED, LED_SMD:LED_0805_2012Metric_Pad1.15x1.40mm_HandSolder, symbol Device:LED
- added R6, R7: 3K, Resistor_SMD:R_1206_3216Metric_Pad1.30x1.75mm_HandSolder, symbol Device:R
- added U10, U7, U9: PCA9745, Package_SO:HTSSOP-28-1EP_4.4x9.7mm_P0.65mm_EP2.85x5.4mm, symbol Project_Library:PCA9745
- added U6: AZ1117-3.3, Package_TO_SOT_SMD:SOT-89-3_Handsoldering, symbol Regulator_Linear:AZ1117-3.3
- D100, D101, D102, D103, D104, D105, D107, D108, D110, D112, D114, D116, D119, D120, D121, D122, D123, D124, D125, D128, D65, D66, D68, D71, D72, D73, D75, D76, D77, D78, D79, D81, D87, D89, D90, D91, D92, D93, D94, D95, D96, D97, D98, D99: renamed from D?; value G_LED -> R_LED
- gave numbers to parts that had none: 7
Connections:
- net EP: now also C7.2, C8.2, R6.2, R7.2, U10.10 (VSS), U10.19 (VSS), U10.2 (VSS), U10.24 (VSS), U10.29 (EP), U6.1 (GND), U7.10 (VSS), U7.19 (VSS), U7.2 (VSS), U7.24 (VSS), U7.29 (EP), U9.10 (VSS), U9.19 (VSS), U9.2 (VSS), U9.24 (VSS), U9.29 (EP)
- net SPI1_CLK: now also U10.26 (SCLK), U7.26 (SCLK), U9.26 (SCLK)
- net SPI1_MISO: now also U10.3 (SDO)
- net SPI1_MOSI: now also U7.27 (SDI)
- net ~OE~: now also U10.5 (~OE~), U7.5 (~OE~), U9.5 (~OE~)
- net ~RESET~: now also U10.25 (~RESET~), U7.25 (~RESET~), U9.25 (~RESET~)
- net at R5.1: now also U7.1 (REXT)
- net at D73.1 (K): now also U7.11 (LED4)
- net at D75.1 (K): now also U7.12 (LED5)
- net at D77.1 (K): now also U7.13 (LED6)
- net at D79.1 (K): now also U7.14 (LED7)
- net at D81.1 (K): now also U7.15 (LED8)
- net at D87.1 (K): now also U7.18 (LED11)
- net at D89.1 (K): now also U7.20 (LED12)
- net at D91.1 (K): now also U7.21 (LED13)
- net at D93.1 (K): now also U7.22 (LED14)
- net at D95.1 (K): now also U7.23 (LED15)
- net at D65.1 (K): now also U7.6 (LED0)
- net at D71.1 (K): now also U7.9 (LED3)
- net at D105.1 (K): now also U9.11 (LED4)
- net at D107.1 (K): now also U9.12 (LED5)
- net at D119.1 (K): now also U9.18 (LED11)
- net at D121.1 (K): now also U9.20 (LED12)
- net at D123.1 (K): now also U9.21 (LED13)
- net at D125.1 (K): now also U9.22 (LED14)
- net at U8.27 (SDI): now also U9.3 (SDO)
- net at D97.1 (K): now also U9.6 (LED0)
- net at D99.1 (K): now also U9.7 (LED1)
- net at D101.1 (K): now also U9.8 (LED2)
- net at D103.1 (K): now also U9.9 (LED3)
- net at U8.1 (REXT): now also R6.1
- net at U8.11 (LED4): now also D74.1 (K)
- net at U8.14 (LED7): now also D80.1 (K)
- net at U8.15 (LED8): now also D82.1 (K)
- net at U8.16 (LED9): now also D84.1 (K)
- net at U8.17 (LED10): now also D86.1 (K)
- net at U8.18 (LED11): now also D88.1 (K)
- net at U8.3 (SDO): now also U10.27 (SDI)
- net at U8.8 (LED2): now also D70.1 (K)
- net at R8.1: now also U10.1 (REXT)
- net at D108.1 (K): now also U10.12 (LED5)
- net at D110.1 (K): now also U10.13 (LED6)
- net at D112.1 (K): now also U10.14 (LED7)
- net at D114.1 (K): now also U10.15 (LED8)
- net at D116.1 (K): now also U10.16 (LED9)
- net at D120.1 (K): now also U10.18 (LED11)
- net at D122.1 (K): now also U10.20 (LED12)
- net at D124.1 (K): now also U10.21 (LED13)
- net at D128.1 (K): now also U10.23 (LED15)
- net at D98.1 (K): now also U10.6 (LED0)
- net at D100.1 (K): now also U10.7 (LED1)
- net at D102.1 (K): now also U10.8 (LED2)
- net at D104.1 (K): now also U10.9 (LED3)
- net +12V renamed R_12V
- net R_12V: now also C7.1, D106.2 (A), D109.2 (A), D111.2 (A), D113.2 (A), D115.2 (A), D117.2 (A), D118.2 (A), D126.2 (A), D127.2 (A), D67.2 (A), D69.2 (A), D70.2 (A), D74.2 (A), D80.2 (A), D82.2 (A), D83.2 (A), D84.2 (A), D85.2 (A), D86.2 (A), D88.2 (A), U6.3 (VI)
- net +3V3 renamed R_3V3
- net R_3V3: now also C8.1, U10.28 (VDD), U6.2 (VO), U7.28 (VDD), U9.28 (VDD)
- net ~CS~_GREEN renamed ~CS~_RED
- net ~CS~_RED: now also U10.4 (~CS~), U7.4 (~CS~), U9.4 (~CS~)
- new net: D83.1 (K), U7.16 (LED9)
- new net: D85.1 (K), U7.17 (LED10)
- new net: U7.3 (SDO), U9.27 (SDI)
- new net: D67.1 (K), U7.7 (LED1)
- new net: D69.1 (K), U7.8 (LED2)
- new net: R7.1, U9.1 (REXT)
- new net: D109.1 (K), U9.13 (LED6)
- new net: D111.1 (K), U9.14 (LED7)
- new net: D113.1 (K), U9.15 (LED8)
- new net: D115.1 (K), U9.16 (LED9)
- new net: D117.1 (K), U9.17 (LED10)
- new net: D127.1 (K), U9.23 (LED15)
- new net: D106.1 (K), U10.11 (LED4)
- new net: D118.1 (K), U10.17 (LED10)
- new net: D126.1 (K), U10.22 (LED14)
Other:
- moved on the sheet: C11, C9, D101, D103, D105, D107, D119, D121, D123, D125, D65, D71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

Commit message: Rev A0 Commit
Files all sent to PCB manufacturer & BOM
Connections:
- net SPI1_MISO: now also U7.3 (SDO); no longer U10.3 (SDO)
- net SPI1_MOSI: now also U10.27 (SDI); no longer U7.27 (SDI)
- net at U8.27 (SDI): now also U10.3 (SDO); no longer U9.3 (SDO)
- net at U8.3 (SDO): now also U9.27 (SDI); no longer U10.27 (SDI)
- new net: U7.27 (SDI), U9.3 (SDO)
Changed lines of the file:
@@
 Wire Wire Line
 	3650 1800 3725 1800
-Text HLabel 3650 1900 0    50   Input ~ 0
+Text HLabel 7850 4650 0    50   Input ~ 0
 SPI1_MOSI
-Wire Wire Line
-	3650 1900 3725 1900
 Text HLabel 3650 2100 0    50   Input ~ 0
 SPI1_CLK
@@
 	7925 4950 7850 4950
 Wire Wire Line
-	3725 2000 2650 2000
-Wire Wire Line
-	2650 2000 2650 4650
-Wire Wire Line
-	2650 4650 3725 4650
-Wire Wire Line
-	3725 4750 2650 4750
-Wire Wire Line
-	2650 4750 2650 6500
-Wire Wire Line
-	2650 6500 6350 6500
-Wire Wire Line
-	6350 6500 6350 1900
-Wire Wire Line
-	6350 1900 7925 1900
-Wire Wire Line
-	7925 2000 6650 2000
-Wire Wire Line
-	6650 2000 6650 4650
-Wire Wire Line
-	7925 4650 6650 4650
-Text HLabel 7850 4750 0    50   Output ~ 0
+	2550 6500 6350 6500
+Wire Wire Line
+	6350 6500 6350 2000
+Text HLabel 3725 2000 0    50   Output ~ 0
 SPI1_MISO
-Wire Wire Line
-	7850 4750 7925 4750
 $Comp
 L Regulator_Linear:AZ1117-3.3 U6
@@
 Text HLabel 10050 3700 1    50   Input ~ 0
 R_12V
+Wire Wire Line
+	2650 1900 3725 1900
+Wire Wire Line
+	6650 4750 7925 4750
+Wire Wire Line
+	7850 4650 7925 4650
+Wire Wire Line
+	6650 1900 7925 1900
+Wire Wire Line
+	6650 1900 6650 4750
+Wire Wire Line
+	7925 2000 6350 2000
+Wire Wire Line
+	2650 4750 3725 4750
+Wire Wire Line
+	2650 1900 2650 4750
+Wire Wire Line
+	3725 4650 2550 4650
+Wire Wire Line
+	2550 4650 2550 6500
 $EndSCHEMATC
