File: LED Wheel/LED Wheel.kicad_pcb (KiCad board)
At the start: 2 copper layers, 60 x 319 mm, 243 parts, among them J1 I/O, J2 I/O, J3 I/O, U1 AZ1117-3.3, U10 PCA9745, U11 AZ1117-3.3, U12 PCA9745, U13 PCA9745, U14 PCA9745, U15 PCA9745, U2 PCA9745, U3 PCA9745, U4 PCA9745, U5 PCA9745, U6 AZ1117-3.3, U7 PCA9745, U8 PCA9745, U9 PCA9745

Commit message: Rev A0 Commit
Files all sent to PCB manufacturer & BOM
Parts:
- added G***: LOGO, Project_Library:pcb_logo, B.Cu at (301.5, 110.5)
- added G***: LOGO, Project_Library:pcb_logo, B.Cu at (301.5, 130.5)
- added G***: LOGO, Project_Library:pcb_logo, B.Cu at (301.5, 150.5)
- moved D129 428.0 mm to (363.0, 116.0), turned to 270 degrees
- moved D131 421.9 mm to (358.0, 116.0), turned to 270 degrees
- moved D133 415.7 mm to (353.0, 116.0), turned to 270 degrees
- moved D1 414.9 mm to (363.0, 136.0), turned to 270 degrees
- moved D135 409.6 mm to (348.0, 116.0), turned to 270 degrees
- moved D3 408.6 mm to (358.0, 136.0), turned to 270 degrees
- moved D137 403.6 mm to (343.0, 116.0), turned to 270 degrees
- moved D65 403.4 mm to (363.0, 156.0), turned to 270 degrees
- moved D5 402.2 mm to (353.0, 136.0), turned to 270 degrees
- moved D139 397.6 mm to (338.0, 116.0), turned to 270 degrees
- moved D67 396.9 mm to (358.0, 156.0), turned to 270 degrees
- moved D7 395.9 mm to (348.0, 136.0), turned to 270 degrees
- moved R9 395.9 mm to (332.4, 109.5), turned to 0 degrees
- moved D141 391.6 mm to (333.0, 116.0), turned to 270 degrees
- moved D69 390.3 mm to (353.0, 156.0), turned to 270 degrees
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Connections:
- net SPI1_CLK renamed /Blue LED Controller/SPI1_CLK
- J1 pad 2: ~CS~_BLUE -> /Blue LED Controller/~OE~
- J1 pad 3: SPI1_MOSI -> /Blue LED Controller/~CS~_BLUE
- J1 pad 4: SPI1_MISO -> /Blue LED Controller/~RESET~
- J1 pad 6: ~0E~ -> /Blue LED Controller/SPI1_MOSI
- J1 pad 7: ~RESET~ -> /Blue LED Controller/SPI1_MISO
- J2 pad 2: ~CS~_RED -> /Blue LED Controller/~OE~
- J2 pad 3: SPI1_MOSI -> /Red LED Controller/~CS~_RED
- J2 pad 4: SPI1_MISO -> /Blue LED Controller/~RESET~
- J2 pad 6: ~0E~ -> /Blue LED Controller/SPI1_MOSI
- J2 pad 7: ~RESET~ -> /Blue LED Controller/SPI1_MISO
- J3 pad 2: ~CS~_GREEN -> /Blue LED Controller/~OE~
- J3 pad 3: SPI1_MOSI -> /Green LED Controller/~CS~_GREEN
- J3 pad 4: SPI1_MISO -> /Blue LED Controller/~RESET~
- J3 pad 6: ~0E~ -> /Blue LED Controller/SPI1_MOSI
- J3 pad 7: ~RESET~ -> /Blue LED Controller/SPI1_MISO
- U10 pad 25: ~RESET~ -> /Blue LED Controller/~RESET~
- U10 pad 27: Net-(U10-Pad27) -> /Blue LED Controller/SPI1_MOSI
- U10 pad 3: SPI1_MISO -> Net-(U10-Pad3)
- U10 pad 4: ~CS~_RED -> /Red LED Controller/~CS~_RED
- U10 pad 5: ~0E~ -> /Blue LED Controller/~OE~
- U12 pad 25: ~RESET~ -> /Blue LED Controller/~RESET~
- U12 pad 27: SPI1_MOSI -> Net-(U12-Pad27)
- U12 pad 3: Net-(U12-Pad3) -> /Blue LED Controller/SPI1_MISO
- U12 pad 4: ~CS~_BLUE -> /Blue LED Controller/~CS~_BLUE
- U12 pad 5: ~0E~ -> /Blue LED Controller/~OE~
- U13 pad 25: ~RESET~ -> /Blue LED Controller/~RESET~
- U13 pad 4: ~CS~_BLUE -> /Blue LED Controller/~CS~_BLUE
- U13 pad 5: ~0E~ -> /Blue LED Controller/~OE~
- U14 pad 25: ~RESET~ -> /Blue LED Controller/~RESET~
- U14 pad 27: Net-(U12-Pad3) -> Net-(U13-Pad3)
- U14 pad 3: Net-(U13-Pad27) -> Net-(U12-Pad27)
- U14 pad 4: ~CS~_BLUE -> /Blue LED Controller/~CS~_BLUE
- U14 pad 5: ~0E~ -> /Blue LED Controller/~OE~
- U15 pad 25: ~RESET~ -> /Blue LED Controller/~RESET~
- U15 pad 27: Net-(U13-Pad3) -> /Blue LED Controller/SPI1_MOSI
- U15 pad 3: SPI1_MISO -> Net-(U13-Pad27)
- U15 pad 4: ~CS~_BLUE -> /Blue LED Controller/~CS~_BLUE
- U15 pad 5: ~0E~ -> /Blue LED Controller/~OE~
- U2 pad 25: ~RESET~ -> /Blue LED Controller/~RESET~
- U2 pad 27: SPI1_MOSI -> Net-(U2-Pad27)
- U2 pad 3: Net-(U2-Pad3) -> /Blue LED Controller/SPI1_MISO
- U2 pad 4: ~CS~_GREEN -> /Green LED Controller/~CS~_GREEN
- U2 pad 5: ~0E~ -> /Blue LED Controller/~OE~
- U3 pad 25: ~RESET~ -> /Blue LED Controller/~RESET~
- U3 pad 4: ~CS~_GREEN -> /Green LED Controller/~CS~_GREEN
- U3 pad 5: ~0E~ -> /Blue LED Controller/~OE~
- U4 pad 25: ~RESET~ -> /Blue LED Controller/~RESET~
- U4 pad 27: Net-(U2-Pad3) -> Net-(U3-Pad3)
- U4 pad 3: Net-(U3-Pad27) -> Net-(U2-Pad27)
- U4 pad 4: ~CS~_GREEN -> /Green LED Controller/~CS~_GREEN
- U4 pad 5: ~0E~ -> /Blue LED Controller/~OE~
- U5 pad 25: ~RESET~ -> /Blue LED Controller/~RESET~
- U5 pad 27: Net-(U3-Pad3) -> /Blue LED Controller/SPI1_MOSI
- U5 pad 3: SPI1_MISO -> Net-(U3-Pad27)
- U5 pad 4: ~CS~_GREEN -> /Green LED Controller/~CS~_GREEN
- U5 pad 5: ~0E~ -> /Blue LED Controller/~OE~
- U7 pad 25: ~RESET~ -> /Blue LED Controller/~RESET~
- U7 pad 27: SPI1_MOSI -> Net-(U7-Pad27)
- U7 pad 3: Net-(U7-Pad3) -> /Blue LED Controller/SPI1_MISO
- U7 pad 4: ~CS~_RED -> /Red LED Controller/~CS~_RED
- U7 pad 5: ~0E~ -> /Blue LED Controller/~OE~
- U8 pad 25: ~RESET~ -> /Blue LED Controller/~RESET~
- U8 pad 27: Net-(U8-Pad27) -> Net-(U10-Pad3)
- U8 pad 3: Net-(U10-Pad27) -> Net-(U8-Pad3)
- U8 pad 4: ~CS~_RED -> /Red LED Controller/~CS~_RED
- U8 pad 5: ~0E~ -> /Blue LED Controller/~OE~
- U9 pad 25: ~RESET~ -> /Blue LED Controller/~RESET~
- U9 pad 27: Net-(U7-Pad3) -> Net-(U8-Pad3)
- U9 pad 3: Net-(U8-Pad27) -> Net-(U7-Pad27)
- U9 pad 4: ~CS~_RED -> /Red LED Controller/~CS~_RED
- U9 pad 5: ~0E~ -> /Blue LED Controller/~OE~
Routing:
- net /Blue LED Controller/~OE~: track 0.00 -> 1225.0 mm, vias 0 -> 12
- net /Blue LED Controller/~RESET~: track 0.00 -> 1072.8 mm, vias 0 -> 9
- net /Blue LED Controller/SPI1_CLK: track 0.00 -> 1062.3 mm, vias 0 -> 9
- net /Blue LED Controller/SPI1_MISO: track 0.00 -> 842.1 mm, vias 0 -> 6
- net /Green LED Controller/~CS~_GREEN: track 0.00 -> 405.3 mm, vias 0 -> 4
- net /Blue LED Controller/~CS~_BLUE: track 0.00 -> 403.7 mm, vias 0 -> 4
- net /Red LED Controller/~CS~_RED: track 0.00 -> 400.4 mm, vias 0 -> 4
- net EP: track 0.00 -> 212.4 mm, vias 0 -> 33
- net Net-(U13-Pad27): track 0.00 -> 75.3 mm
- net Net-(U12-Pad27): track 0.00 -> 74.7 mm
- net Net-(U13-Pad3): track 0.00 -> 74.5 mm
- net Net-(U8-Pad3): track 0.00 -> 74.5 mm
- net Net-(U7-Pad27): track 0.00 -> 74.5 mm
- net Net-(U3-Pad3): track 0.00 -> 74.5 mm
- net Net-(U3-Pad27): track 0.00 -> 74.5 mm
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Other:
- board size 60 x 319 mm -> 325 x 60 mm
- board text added: "12V+"
- board text added: "GND"
- board text added: "LED Wheel Display Rev. A0"
- board text added: "SPI_CLK"
- board text added: "SPI_MISO"
- board text added: "SPI_MOSI"
- board text added: "nCS_BLUE"
- board text added: "nCS_GREEN"
- board text added: "nCS_RED"
- board text added: "nOE"
- board text added: "nRESET"

Commit message: Updated LED Wheel for PCBWay
Added Light reflector for speed sensor, updated board layout for VCut
Parts:
- added J4: G_12V, Connector_PinHeader_2.54mm:PinHeader_1x01_P2.54mm_Vertical, B.Cu at (49.0, 140.0)
- added J5: R_12V, Connector_PinHeader_2.54mm:PinHeader_1x01_P2.54mm_Vertical, B.Cu at (49.0, 160.0)
- added J6: B_12V, Connector_PinHeader_2.54mm:PinHeader_1x01_P2.54mm_Vertical, B.Cu at (49.0, 120.0)
- added TP1: Reflector, Project_Library:Reflector 2x4mm, F.Cu at (125.5, 160.5)
- added TP2: Reflector, Project_Library:Reflector 2x4mm, F.Cu at (125.5, 140.5)
- added TP3: Reflector, Project_Library:Reflector 2x4mm, F.Cu at (125.5, 120.5)
Routing:
- net +12V: track 14.5 -> 0.00 mm, vias 3 -> 6
- added copper zone on B.Cu, net +12V
Other:
- board size 325 x 60 mm -> 325 x 80 mm
